File: pcb/ble.kicad_sch (KiCad schematic)
At the start: 9 parts, among them J5 Conn_ARM_SWD_TagConnect_TC203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, U9 BLUENRG-M2SP

Commit message: update
Connections:
- no-connect marks 12 -> 14
Other:
- moved on the sheet: C26, C27, C28, J5, JP2, JP3, JP4, JP5, U9
