File: pcb/pcb.kicad_sch (KiCad schematic)
At the start: 22 parts, among them J1 Conn_ARM_SWD_TagConnect_TC2030, SW1 RESET_BUTTON, U1 STM32G431KBTx, Y1 830103622909

Commit message: update
Parts:
- added G1: LOGO, custom:logo, symbol custom:LOGO
- J1: value Conn_ARM_SWD_TagConnect_TC2030 -> Conn_ARM_SWD_TagConnect_TC2030-NL; footprint Connector:Tag-Connect_TC2030-IDC-FP_2x03_P1.27mm_Vertical -> Connector:Tag-Connect_TC2030-IDC-NL_2x03_P1.27mm_Vertical
Other:
- moved on the sheet: C1, C2, C3, C4, C5, DS1, DS2, DS3, JP1, R1, R2, R4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
