File: pcb/usb.kicad_sch (KiCad schematic)
At the start: 21 parts, among them J2 USB_C_Receptacle_USB2.0_16P, U2 USBLC6-2SC6, U3 FT230XS, U4 SPX3819M5-L, U5 LM66100DCK

Commit message: update
Changed lines of the file:
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@@
-	)
-	(junction
-		(at 114.3 93.98)
-		(diameter 0)
-		(color 0 0 0 0)
 	)
 	(junction
@@
 	(wire
 		(pts
-			(xy 114.3 93.98) (xy 115.57 93.98)
-		)
-		(stroke
-			(width 0)
-			(type default)
-		)
-	)
-	(wire
-		(pts
 			(xy 204.47 49.53) (xy 204.47 52.07)
 		)
@@
 	(wire
 		(pts
-			(xy 100.33 93.98) (xy 114.3 93.98)
+			(xy 100.33 93.98) (xy 115.57 93.98)
 		)
 		(stroke
@@
 	(wire
 		(pts
-			(xy 114.3 93.98) (xy 114.3 97.79)
+			(xy 115.57 93.98) (xy 115.57 97.79)
 		)
 		(stroke
@@
 	(symbol
 		(lib_id "power:GND")
-		(at 114.3 97.79 0)
+		(at 115.57 97.79 0)
 		(unit 1)
 		(exclude_from_sim no)
@@
 		(dnp no)
 		(property "Reference" "#PWR017"
-			(at 114.3 104.14 0)
+			(at 115.57 104.14 0)
 			(effects
 				(font
@@
 		)
 		(property "Value" "GND"
-			(at 118.11 99.568 0)
+			(at 119.38 99.568 0)
 			(effects
 				(font
@@
 		)
 		(property "Footprint" ""
-			(at 114.3 97.79 0)
+			(at 115.57 97.79 0)
 			(effects
 				(font
@@
 		)
 		(property "Datasheet" ""
-			(at 114.3 97.79 0)
+			(at 115.57 97.79 0)
 			(effects
 				(font
@@
 		)
 		(property "Description" "Power symbol creates a global label with name \"GND\" , ground"
-			(at 114.3 97.79 0)
-			(effects
-				(font
+			(at 115.57 97.79 0)
+			(effects
+				(font
